Commit message: last

File: urdf/phantomx.urdf (robot description, URDF)
Before this commit: robot PhantomX, 28 links, 27 joints
Links:
- added link base_scan, mass 0.114; collision cylinder length=0.0315 radius=0.055; visual mesh filename=package://phantomx_description/meshes/lds.stl scale=0.001 0.001 0.001
Joints:
- added joint scan_joint: type fixed, parent base_link, child base_scan, origin xyz=-0.0 0 0.05 rpy=0 0 0
